Commit message: Add modules for simulating airship software pipeline in Nvidia Isaac.

File: airship_description/urdf/airsbot2.urdf (robot description, URDF)
Before this commit: robot airsbot2, 3 links, 2 joints
Links:
- added link base, mass 0.01; collision mesh filename=package://airship_description/urdf/meshes//arm_base.stl scale=0.001 0.001 0.001; visual mesh filename=package://airship_description/urdf/meshes//arm_base.stl scale=0.001 0.001 0.001
- added link base_footprint
- added link camera_support_link, mass 0.05; collision mesh filename=package://airship_description/urdf/meshes/camera_base.stl scale=0.001 0.001 0.001; visual mesh filename=package://airship_description/urdf/meshes/camera_base.stl scale=0.001 0.001 0.001
- added link carrier_link, mass 0.1; collision mesh filename=package://airship_description/urdf/meshes/carrier.stl scale=0.001 0.001 0.001; visual mesh filename=package://airship_description/urdf/meshes/carrier.stl scale=0.001 0.001 0.001
- added link ee_link
- added link front_camera_link
- added link gripper_base, mass 0.05; collision mesh filename=package://airship_description/urdf/meshes/gripper_base.stl scale=0.001 0.001 0.001; visual mesh filename=package://airship_description/urdf/meshes/gripper_base.stl scale=0.001 0.001 0.001
- added link gripper_camera_link; visual mesh filename=package://airship_description/urdf/meshes/IntelRealsense_D4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 scale=0.001 0.001 0.001
- added link gripper_left1, mass 0.05; collision mesh filename=package://airship_description/urdf/meshes/gripper_left1.stl scale=0.001 0.001 0.001; visual mesh filename=package://airship_description/urdf/meshes/gripper_left1.stl scale=0.001 0.001 0.001
- added link gripper_left2, mass 0.05; collision mesh filename=package://airship_description/urdf/meshes/gripper_left2.stl scale=0.001 0.001 0.001; visual mesh filename=package://airship_description/urdf/meshes/gripper_left2.stl scale=0.001 0.001 0.001
- added link gripper_left3, mass 0.05; collision mesh filename=package://airship_description/urdf/meshes/gripper_left3.stl scale=0.001 0.001 0.001; visual mesh filename=package://airship_description/urdf/meshes/gripper_left3.stl scale=0.001 0.001 0.001
- added link gripper_right1, mass 0.05; collision mesh filename=package://airship_description/urdf/meshes/gripper_right1.stl scale=0.001 0.001 0.001; visual mesh filename=package://airship_description/urdf/meshes/gripper_right1.stl scale=0.001 0.001 0.001
- added link gripper_right2, mass 0.05; collision mesh filename=package://airship_description/urdf/meshes/gripper_right2.stl scale=0.001 0.001 0.001; visual mesh filename=package://airship_description/urdf/meshes/gripper_right2.stl scale=0.001 0.001 0.001
- added link gripper_right3, mass 0.05; collision mesh filename=package://airship_description/urdf/meshes/gripper_right3.stl scale=0.001 0.001 0.001; visual mesh filename=package://airship_description/urdf/meshes/gripper_right3.stl scale=0.001 0.001 0.001
- added link left_back_driven_wheel_link, mass 7.15; collision cylinder length=0.075 radius=0.120; visual mesh filename=package://airship_description/urdf/meshes/wheel.stl scale=0.001 0.001 0.001
- added link left_driving_wheel_link, mass 7.15; collision cylinder length=0.075 radius=0.1205
- added link left_front_driven_wheel_link, mass 7.15; collision cylinder length=0.075 radius=0.120; visual mesh filename=package://airship_description/urdf/meshes/wheel.stl scale=0.001 0.001 0.001
- added link lidar_link, mass 0.5; collision mesh filename=package://airship_description/urdf/meshes/Helios_Lede_20220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 scale=0.001 0.001 0.001; visual mesh filename=package://airship_description/urdf/meshes/Helios_Lede_20220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 scale=0.001 0.001 0.001
- added link link1, mass 0.01; collision mesh filename=package://airship_description/urdf/meshes//link1.stl scale=0.001 0.001 0.001; visual mesh filename=package://airship_description/urdf/meshes//link1.stl scale=0.001 0.001 0.001
- added link link2, mass 0.01; collision mesh filename=package://airship_description/urdf/meshes//link2.stl scale=0.001 0.001 0.001; visual mesh filename=package://airship_description/urdf/meshes//link2.stl scale=0.001 0.001 0.001
- added link link3, mass 0.01; collision mesh filename=package://airship_description/urdf/meshes//link3.stl scale=0.001 0.001 0.001; visual mesh filename=package://airship_description/urdf/meshes//link3.stl scale=0.001 0.001 0.001
- added link link4, mass 0.01; collision mesh filename=package://airship_description/urdf/meshes//link4.stl scale=0.001 0.001 0.001; visual mesh filename=package://airship_description/urdf/meshes//link4.stl scale=0.001 0.001 0.001
- added link link5, mass 0.01; collision mesh filename=package://airship_description/urdf/meshes//link5.stl scale=0.001 0.001 0.001; visual mesh filename=package://airship_description/urdf/meshes//link5.stl scale=0.001 0.001 0.001
- added link link6, mass 0.01; collision mesh filename=package://airship_description/urdf/meshes//link6.stl scale=0.001 0.001 0.001; visual mesh filename=package://airship_description/urdf/meshes//link6.stl scale=0.001 0.001 0.001
- added link manipulator_base_link, mass 0.1; collision mesh filename=package://airship_description/urdf/meshes/manipulator_base.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 scale=0.001 0.001 0.001; visual mesh filename=package://airship_description/urdf/meshes/manipulator_base.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 scale=0.001 0.001 0.001
- added link right_back_driven_wheel_link, mass 7.15; collision cylinder length=0.075 radius=0.120; visual mesh filename=package://airship_description/urdf/meshes/wheel.stl scale=0.001 0.001 0.001
- added link right_driving_wheel_link, mass 7.15; collision cylinder length=0.075 radius=0.1205
- added link right_front_driven_wheel_link, mass 7.15; collision cylinder length=0.075 radius=0.120; visual mesh filename=package://airship_description/urdf/meshes/wheel.stl scale=0.001 0.001 0.001
- added link sensor_d435_bottom_screw_frame
- added link sensor_d435_color_frame
- added link sensor_d435_color_optical_frame
- added link sensor_d435_depth_frame
- added link sensor_d435_depth_optical_frame
- added link sensor_d435_left_ir_frame
- added link sensor_d435_left_ir_optical_frame
- added link sensor_d435_link, mass 0.0564
- added link sensor_d435_right_ir_frame
- added link sensor_d435_right_ir_optical_frame
- added link zed2_baro_link
- added link zed2_camera_center
- added link zed2_camera_link, mass 0.0564; visual mesh filename=package://airship_description/urdf/meshes/ZED2.stl scale=0.001 0.001 0.001
- added link zed2_left_camera_frame
- added link zed2_left_camera_optical_frame
- added link zed2_mag_link
- added link zed2_right_camera_frame
- added link zed2_right_camera_optical_frame
- added link zed2_temp_left_link
- added link zed2_temp_right_link
- link base_link: mass None -> 30.0; geometry collision box size=0.7 0.588 0.056; visual box size=0.7 0.588 0.056
Joints:
- removed joint imu_link_joint
- removed joint rslidar_joint
- added joint base_joint: type fixed, parent base_footprint, child base_link, origin xyz=0.0 0.0 0.309 rpy=0.0 0.0 0.0
- added joint camera_support_to_gripper_base_joint: type fixed, parent camera_support_link, child gripper_base, origin xyz=0.0485 -0.002 0.007 rpy=0.0 0.0 -1.5707963267948966
- added joint carrier_joint: type fixed, parent base_link, child carrier_link, origin xyz=0.255 0.0 0.033 rpy=0.0 0.0 0.0
- added joint gripper_base_to_gripper_left2: type revolute, parent gripper_base, child gripper_left2, origin xyz=-0.05 -0.01 0 rpy=0.0 0.0 0.0, axis 0.0 0.0 1.0, limit lower=-0.8 upper=0.5 effort=1000.0 velocity=0.0, mimic joint=gripper_controller multiplier=1.0 offset=0.0
- added joint gripper_base_to_gripper_right2: type revolute, parent gripper_base, child gripper_right2, origin xyz=0.046 -0.01 0.0 rpy=0.0 0.0 0.0, axis 0.0 0.0 1.0, limit lower=-0.5 upper=0.8 effort=1000.0 velocity=0.0, mimic joint=gripper_controller multiplier=-1.0 offset=0.0
- added joint gripper_base_to_gripper_right3: type revolute, parent gripper_base, child gripper_right3, origin xyz=0.018 0.016 0.0 rpy=0.0 0.0 0.0, axis 0.0 0.0 1.0, limit lower=-0.3 upper=0.7 effort=1000.0 velocity=0, mimic joint=gripper_controller multiplier=-1.0 offset=0.0
- added joint gripper_camera_joint: type fixed, parent camera_support_link, child gripper_camera_link, origin xyz=0.042 0 0.048 rpy=0.0 0.0 0.0
- added joint gripper_controller: type revolute, parent gripper_base, child gripper_left3, origin xyz=-0.018 0.016 0.0 rpy=0.0 0.0 0.0, axis 0.0 0.0 1.0, limit lower=-0.7 upper=0.3 effort=1000.0 velocity=0.0
- added joint gripper_joint: type fixed, parent ee_link, child camera_support_link, origin xyz=0.0 0.0 0.0 rpy=0.0 0.0 0.0
- added joint gripper_left3_to_gripper_left1: type revolute, parent gripper_left3, child gripper_left1, origin xyz=-0.0356 0.051 -0.018 rpy=0.0 0.0 0.0, axis 0.0 0.0 1.0, limit lower=-0.5 upper=0.5 effort=1000.0 velocity=0.0, mimic joint=gripper_controller multiplier=-1.0 offset=0.0
- added joint gripper_right3_to_gripper_right1: type revolute, parent gripper_right3, child gripper_right1, origin xyz=0.033 0.051 -0.018 rpy=0.0 0.0 0.0, axis 0.0 0.0 1.0, limit lower=-0.5 upper=0.5 effort=1000.0 velocity=0.0, mimic joint=gripper_controller multiplier=1.0 offset=0.0
- added joint imu_joint: type fixed, parent base_link, child imu_link, origin xyz=0.255 0.0 0.033 rpy=0.0 0.0 0.0
- added joint joint_base_to_manipulator_base_link: type fixed, parent manipulator_base_link, child base, origin xyz=0.0 0.0 0.0 rpy=0.0 0.0 0.0
- added joint joint_ee_link_to_link6: type fixed, parent link6, child ee_link, origin xyz=0.0 0.0 0.0 rpy=2.748893571891069 0 3.141592653589793
- added joint joint_link1_to_base: type revolute, parent base, child link1, origin xyz=0.0 0.0 0.22934 rpy=0.0 0.0 0.0, axis 0.0 0.0 1.0, limit lower=-3.141592653589793 upper=3.141592653589793 effort=1000.0 velocity=0
- added joint joint_link2_to_link1: type revolute, parent link1, child link2, origin xyz=0.0 0.0 0.0 rpy=1.5707963267948966 0.0 0.0, axis 0.0 0.0 -1.0, limit lower=-4.71238898038469 upper=1.5707963267948966 effort=1000.0 velocity=0.0
- added joint joint_link3_to_link2: type revolute, parent link2, child link3, origin xyz=0.27 0.0 0.0 rpy=0.0 0.0 0.0, axis 0.0 0.0 -1.0, limit lower=-2.607521902479528 upper=2.607521902479528 effort=1000.0 velocity=0.0
- added joint joint_link4_to_link3: type revolute, parent link3, child link4, origin xyz=0.267 0.0 -0.0745 rpy=0.0 0.0 0.0, axis 0.0 0.0 -1.0, limit lower=-4.523893421169302 upper=1.382300767579509 effort=1000.0 velocity=0.0
- added joint joint_link5_to_link4: type revolute, parent link4, child link5, origin xyz=0.0 -0.095 0.002 rpy=1.5707963267948966 -1.5707963267948966 0.0, axis 0.0 0.0 1.0, limit lower=-2.921681167838508 upper=2.921681167838508 effort=1000.0 velocity=0.0
- added joint joint_link6_to_link5: type revolute, parent link5, child link6, origin xyz=-0.054 0.0 0.0 rpy=-1.5707963267948966 0.0 0.0, axis -1.0 0.0 0.0, limit lower=-3.015928947446201 upper=3.015928947446201 effort=1000.0 velocity=0
- added joint left_back_driven_wheel_joint: type continuous, parent base_link, child left_back_driven_wheel_link, origin xyz=-0.23 0.219 -0.182 rpy=-1.5707963267948966 0.0 0.0, axis 0.0 0.0 1.0, limit lower=-1e+16 upper=1e+16 effort=25.0 velocity=75.36
- added joint left_driving_wheel_joint: type continuous, parent base_link, child left_driving_wheel_link, origin xyz=0.0 0.219 -0.182 rpy=-1.5707963267948966 0.0 0.0, axis 0.0 0.0 1.0, limit lower=-1e+16 upper=1e+16 effort=25.0 velocity=75.36
- added joint left_front_driven_wheel_joint: type continuous, parent base_link, child left_front_driven_wheel_link, origin xyz=0.23 0.219 -0.182 rpy=-1.5707963267948966 0.0 0.0, axis 0.0 0.0 1.0, limit lower=-1e+16 upper=1e+16 effort=25.0 velocity=75.36
- added joint lidar_joint: type fixed, parent base_link, child lidar_link, origin xyz=0.255 0.0 0.156 rpy=0.0 0.0 0.0
- added joint lidar_optical_joint: type fixed, parent lidar_link, child rslidar, origin xyz=0.0 0.0 0.0 rpy=0.0 0.0 0.0
- added joint manipulator_base_joint: type fixed, parent base_link, child manipulator_base_link, origin xyz=0.255 0.0 0.262 rpy=0.0 0.0 0.0
- added joint right_back_driven_wheel_joint: type continuous, parent base_link, child right_back_driven_wheel_link, origin xyz=-0.23 -0.219 -0.182 rpy=-1.5707963267948966 0.0 0.0, axis 0.0 0.0 1.0, limit lower=-1e+16 upper=1e+16 effort=25.0 velocity=75.36
- added joint right_driving_wheel_joint: type continuous, parent base_link, child right_driving_wheel_link, origin xyz=0.0 -0.219 -0.182 rpy=-1.5707963267948966 0.0 0.0, axis 0.0 0.0 1.0, limit lower=-1e+16 upper=1e+16 effort=25.0 velocity=75.36
- added joint right_front_driven_wheel_joint: type continuous, parent base_link, child right_front_driven_wheel_link, origin xyz=0.23 -0.219 -0.182 rpy=-1.5707963267948966 0.0 0.0, axis 0.0 0.0 1.0, limit lower=-1e+16 upper=1e+16 effort=25.0 velocity=75.36
- added joint sensor_d435_color_joint: type fixed, parent sensor_d435_depth_frame, child sensor_d435_color_frame, origin xyz=0 0.015 0 rpy=0 0 0
- added joint sensor_d435_color_optical_joint: type fixed, parent sensor_d435_color_frame, child sensor_d435_color_optical_frame, origin xyz=0 0 0 rpy=-1.5707963267948966 0 -1.5707963267948966
- added joint sensor_d435_depth_joint: type fixed, parent sensor_d435_link, child sensor_d435_depth_frame, origin xyz=0 0 0 rpy=0 0 0
- added joint sensor_d435_depth_optical_joint: type fixed, parent sensor_d435_depth_frame, child sensor_d435_depth_optical_frame, origin xyz=0 0 0 rpy=-1.5707963267948966 0 -1.5707963267948966
- added joint sensor_d435_joint: type fixed, parent gripper_camera_link, child sensor_d435_bottom_screw_frame, origin xyz=0 0 0 rpy=0 0 0
- added joint sensor_d435_left_ir_joint: type fixed, parent sensor_d435_depth_frame, child sensor_d435_left_ir_frame, origin xyz=0 0.0 0 rpy=0 0 0
- added joint sensor_d435_left_ir_optical_joint: type fixed, parent sensor_d435_left_ir_frame, child sensor_d435_left_ir_optical_frame, origin xyz=0 0 0 rpy=-1.5707963267948966 0 -1.5707963267948966
- added joint sensor_d435_link_joint: type fixed, parent sensor_d435_bottom_screw_frame, child sensor_d435_link, origin xyz=0 0.0175 0.0125 rpy=0 0 0
- added joint sensor_d435_right_ir_joint: type fixed, parent sensor_d435_depth_frame, child sensor_d435_right_ir_frame, origin xyz=0 -0.05 0 rpy=0 0 0
- added joint sensor_d435_right_ir_optical_joint: type fixed, parent sensor_d435_right_ir_frame, child sensor_d435_right_ir_optical_frame, origin xyz=0 0 0 rpy=-1.5707963267948966 0 -1.5707963267948966
- added joint zed2_baro_joint: type fixed, parent zed2_camera_center, child zed2_baro_link, origin xyz=0 0 0 rpy=0 0 0
- added joint zed2_camera_center_joint: type fixed, parent zed2_camera_link, child zed2_camera_center, origin xyz=0 0 0.015 rpy=0 0.05 0
- added joint zed2_camera_joint: type fixed, parent front_camera_link, child zed2_camera_link, origin xyz=0 0 0 rpy=0 0 0
- added joint zed2_left_camera_joint: type fixed, parent zed2_camera_center, child zed2_left_camera_frame, origin xyz=-0.01 0.06 0 rpy=0 0 0
- added joint zed2_left_camera_optical_joint: type fixed, parent zed2_left_camera_frame, child zed2_left_camera_optical_frame, origin xyz=0 0 0 rpy=-1.5707963267948966 0.0 -1.5707963267948966
- added joint zed2_mag_joint: type fixed, parent zed2_camera_center, child zed2_mag_link, origin xyz=0 0 0 rpy=0 0 0
- added joint zed2_right_camera_joint: type fixed, parent zed2_camera_center, child zed2_right_camera_frame, origin xyz=-0.01 -0.06 0 rpy=0 0 0
- added joint zed2_right_camera_optical_joint: type fixed, parent zed2_right_camera_frame, child zed2_right_camera_optical_frame, origin xyz=0 0 0 rpy=-1.5707963267948966 0.0 -1.5707963267948966
- added joint zed2_temp_left_joint: type fixed, parent zed2_left_camera_frame, child zed2_temp_left_link, origin xyz=0 0 0 rpy=0 0 0
- added joint zed2_temp_right_joint: type fixed, parent zed2_right_camera_frame, child zed2_temp_right_link, origin xyz=0 0 0 rpy=0 0 0
- added joint zed_camera_joint: type fixed, parent base_link, child front_camera_link, origin xyz=0.320 0.0 0.203 rpy=0.0 0.0 0.0
